File: power_and_monotoring/feather.kicad_sch (KiCad schematic)
At the start: 24 parts, among them U11 CD4051BM96G3, U12 CD4051BM96G3

Commit message: Final
Parts:
- removed R7 (x6): CRCW0805, UniSA_Motorsport_Resistor:0805, symbol UniSA_Motorsport_Resistor:CRCW0805
- added D28, D29, D30, D31: MMBZ5225BS-7-F, UniSA_Motorsport_SOT_TO:SOT-363, symbol UniSA_Motorsport_Diode:MMBZ5225BS-7-F
- added R1, R2, R8: CRCW0805, UniSA_Motorsport_Resistor:0805, symbol UniSA_Motorsport_Resistor:CRCW0805
- added RN1, RN2: EXB-38V103JV, UniSA_Motorsport_Resistor:EXB38V472JV, symbol UniSA_Motorsport_Resistor:EXB-38V103JV
- renumbered R7 to R44, R7 to R45, R7 to R46, R7 to R47, R7 to R48, R7 to R49
Connections:
- net +3V3: now also R1.1, R2.1, R8.1
- net BRAKE_LIGHT_SIG: now also RN2.4; no longer U11.4 (X7)
- net BRAKE_SIG_AMP_HIGH: now also RN1.1; no longer U11.15 (X2)
- net BRAKE_SIG_AMP_SHORT_GND: now also RN2.3; no longer U11.2 (X6)
- net BRAKE_SIG_AMP_SHORT_HIGH: now also RN2.2; no longer U11.5 (X5)
- net GND: now also D28.1 (A), D28.4 (A), D29.1 (A), D29.4 (A), D30.1 (A), D30.4 (A), D31.1 (A), D31.4 (A)
- net POWER_SIG_HIGH: now also RN1.2; no longer U11.14 (X1)
- net POWER_SIG_SHORT_GND: now also RN2.1; no longer U11.1 (X4)
- net POWER_SIG_SHORT_HIGH: now also RN1.4; no longer U11.12 (X3)
- net Sensor_1_Temp: now also TEMP_1.1, U12.13 (X0), R1.2
- net Sensor_2_Temp: now also TEMP_2.1, U12.14 (X1), R8.2
- net Sensor_3_Temp: now also TEMP_3.1, U12.15 (X2), R2.2
- net D_BSPD_TRIGGER: no longer names the net of U11.13 (X0)
- net D_BSPD_TRIGGER: now also D28.3 (K), RN1.8
- new net: D31.6 (K), RN2.5, U11.4 (X7)
- new net: D31.3 (K), RN2.6, U11.2 (X6)
- new net: D30.6 (K), RN2.7, U11.5 (X5)
- new net: D30.3 (K), RN2.8, U11.1 (X4)
- new net: D29.6 (K), RN1.5, U11.12 (X3)
- new net: D28.6 (K), RN1.7, U11.14 (X1)
- new net: D29.3 (K), RN1.6, U11.15 (X2)
- new net BSPD_TRIGGER: RN1.3
Other:
- moved on the sheet: C18, U11
