File: power_and_monotoring/fuses.kicad_sch (KiCad schematic)
At the start: 47 parts, among them K1 G5Q-1A, K2 G5Q-1A, K3 G5Q-1A

Commit message: first connections done (not perfect yet)
Parts:
- R24, R25, R26, R27, R28, R31, R32, R33, R34, R36, R37, R38: footprint Resistor_SMD:R_0805_2012Metric -> UniSA_Motorsport_Resistor:0805
Changed lines of the file:
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@@
       (effects (font (size 1.27 1.27)) (justify left))
     )
-    (property "Footprint" "Resistor_SMD:R_0805_2012Metric" (at 58.039 115.316 90)
+    (property "Footprint" "UniSA_Motorsport_Resistor:0805" (at 58.039 115.316 90)
       (effects (font (size 1.27 1.27)) hide)
     )
@@
       (effects (font (size 1.27 1.27)) (justify left))
     )
-    (property "Footprint" "Resistor_SMD:R_0805_2012Metric" (at 160.909 67.056 90)
+    (property "Footprint" "UniSA_Motorsport_Resistor:0805" (at 160.909 67.056 90)
       (effects (font (size 1.27 1.27)) hide)
     )
@@
       (effects (font (size 1.27 1.27)) (justify left))
     )
-    (property "Footprint" "Resistor_SMD:R_0805_2012Metric" (at 320.421 173.228 90)
+    (property "Footprint" "UniSA_Motorsport_Resistor:0805" (at 320.421 173.228 90)
       (effects (font (size 1.27 1.27)) hide)
     )
@@
       (effects (font (size 1.27 1.27)) (justify left))
     )
-    (property "Footprint" "Resistor_SMD:R_0805_2012Metric" (at 58.039 139.446 90)
+    (property "Footprint" "UniSA_Motorsport_Resistor:0805" (at 58.039 139.446 90)
       (effects (font (size 1.27 1.27)) hide)
     )
@@
       (effects (font (size 1.27 1.27)) (justify left))
     )
-    (property "Footprint" "Resistor_SMD:R_0805_2012Metric" (at 58.039 42.926 90)
+    (property "Footprint" "UniSA_Motorsport_Resistor:0805" (at 58.039 42.926 90)
       (effects (font (size 1.27 1.27)) hide)
     )
@@
       (effects (font (size 1.27 1.27)) (justify left))
     )
-    (property "Footprint" "Resistor_SMD:R_0805_2012Metric" (at 160.909 91.186 90)
+    (property "Footprint" "UniSA_Motorsport_Resistor:0805" (at 160.909 91.186 90)
       (effects (font (size 1.27 1.27)) hide)
     )
@@
       (effects (font (size 1.27 1.27)) (justify left))
     )
-    (property "Footprint" "Resistor_SMD:R_0805_2012Metric" (at 329.946 112.014 90)
+    (property "Footprint" "UniSA_Motorsport_Resistor:0805" (at 329.946 112.014 90)
       (effects (font (size 1.27 1.27)) hide)
     )
@@
       (effects (font (size 1.27 1.27)) (justify left))
     )
-    (property "Footprint" "Resistor_SMD:R_0805_2012Metric" (at 320.421 225.679 90)
+    (property "Footprint" "UniSA_Motorsport_Resistor:0805" (at 320.421 225.679 90)
       (effects (font (size 1.27 1.27)) hide)
     )
@@
       (effects (font (size 1.27 1.27)) (justify left))
     )
-    (property "Footprint" "Resistor_SMD:R_0805_2012Metric" (at 58.039 67.056 90)
+    (property "Footprint" "UniSA_Motorsport_Resistor:0805" (at 58.039 67.056 90)
       (effects (font (size 1.27 1.27)) hide)
     )
@@
       (effects (font (size 1.27 1.27)) (justify left))
     )
-    (property "Footprint" "Resistor_SMD:R_0805_2012Metric" (at 299.339 60.071 90)
+    (property "Footprint" "UniSA_Motorsport_Resistor:0805" (at 299.339 60.071 90)
       (effects (font (size 1.27 1.27)) hide)
     )
@@
       (effects (font (size 1.27 1.27)) (justify left))
     )
-    (property "Footprint" "Resistor_SMD:R_0805_2012Metric" (at 58.039 91.186 90)
+    (property "Footprint" "UniSA_Motorsport_Resistor:0805" (at 58.039 91.186 90)
       (effects (font (size 1.27 1.27)) hide)
     )
@@
       (effects (font (size 1.27 1.27)) (justify left))
     )
-    (property "Footprint" "Resistor_SMD:R_0805_2012Metric" (at 301.244 32.766 90)
-      (effects (font (size 1.27 1.27)) hide)
-    )
+    (property "Footprint" "UniSA_Motorsport_Resistor:0805" (at 301.244 32.766 90)
+      (effects (font (size 1.27 1.27)) hide)
+    )

Commit message: before design review
Parts:
- removed LED10, LED12, LED13, LED14, LED15, LED16, LED17, LED18, LED19, LED20, LED21, LED22, LED23, LED9: GREEN, LTST-S270KGKT, UniSA_Motorsport_Diode:0605, symbol UniSA_Motorsport_Diode:LTST-S270KGKT
- added D5 (x14): GREEN, UniSA_Motorsport_Diode:0805, symbol UniSA_Motorsport_Diode:LED_0805
- added J7: 43045-1615, UniSA_Motorsport_Connector:MOLEX_43045-16YY_16PIN, symbol UniSA_Motorsport_Connector:43045-1615
Connections:
- net +24V: now also J7.1 (Pin_1)
- net 12V_MOTOR_CONTROLLER: now also J7.13 (Pin_13)
- net 24V_RADIATOR_FAN: now also J7.12 (Pin_12)
- net 24V_RADIATOR_PUMP: now also J7.11 (Pin_11)
- net AIR_POWER_24V: now also J7.2 (Pin_2)
- net BREAK_LIGHT_12V: now also J7.9 (Pin_9)
- net BSPD_12V: now also J7.10 (Pin_10)
- net DASH_24V: now also J7.6 (Pin_6)
- net ECU_24V: now also J7.7 (Pin_7)
- net GND: now also D5.1 (K), D5.1 (K), D5.1 (K), D5.1 (K), D5.1 (K), D5.1 (K), D5.1 (K), D5.1 (K), D5.1 (K), D5.1 (K), D5.1 (K), D5.1 (K), D5.1 (K), D5.1 (K), J7.14 (Pin_14), J7.15 (Pin_15), J7.16 (Pin_16)
- net HIGH_VOLTAGE_BOX_24V: now also J7.8 (Pin_8)
- net MASTER_ACCUMULATOR_24V: now also J7.4 (Pin_4)
- net SAFETY_24V: now also J7.3 (Pin_3)
- net SLAVE_ACCUMULATOR_24V: now also J7.5 (Pin_5)
- net at R36.2: now also D5.2 (A)
- net at R27.2: now also D5.2 (A)
- net at R31.2: now also D5.2 (A)
- net at R24.2: now also D5.2 (A)
- net at R37.2: now also D5.2 (A)
- net at R25.2: now also D5.2 (A)
- net at R28.2: now also D5.2 (A)
- net at R26.2: now also D5.2 (A)
- net at R22.2: now also D5.2 (A)
- net at R32.2: now also D5.2 (A)
- net at R39.2: now also D5.2 (A)
- net at R38.2: now also D5.2 (A)
- net at R34.2: now also D5.2 (A)
- net at R33.2: now also D5.2 (A)

Commit message: Final
Parts:
- added D24, D25, D26: 1N4148W RHG, UniSA_Motorsport_Diode:SOD-123F-2, symbol UniSA_Motorsport_Diode:1N4148W_RHG
- R22, R39: Resistance 68K -> 1K
- renumbered TP1 to 24V2, D5 to D10, D5 to D12, D5 to D13, D5 to D14, D5 to D15, D5 to D16, D5 to D17, D5 to D18, D5 to D19, D5 to D20, D5 to D21, D5 to D22, D5 to D23, D5 to D9, TP1 to GLV_IN1, TP1 to GND1
Connections:
- net +24V: now also D24.1 (K), D25.1 (K), D26.1 (K)
- net MOTOR_CONTROLLER_ON_SIGNAL: now also D26.2 (A)
- net PUMP_ON_SIGNAL: now also D24.2 (A)
- net RADIATOR_FAN_ON_SIGNAL: now also D25.2 (A)
Other:
- moved on the sheet: D22, F14, K2, R37

Commit message: Made it 4 layers
Parts:
- R22, R39: Resistance 1K -> 10k
- R24, R25, R26, R27, R28, R31, R32, R33, R34, R36, R37, R38: Resistance 1k -> 10k
Connections:
- net +12V: now also F2.1
- net +24V: no longer F2.1
- net PUMP_FUSE_RELAY: now reaches F13.2, K1.3
- net SAFETY_24V renamed SAFETY_12V
Other:
- moved on the sheet: D13, D21, D22, D23, D24, D25, D26, F13, F14, F15, F2, GND1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
